Commit message: change fix bug

File: description/robot_core.xacro (robot description, xacro)
@@ -32,5 +32,5 @@
         <parent link="base_link"/>
         <child link="chassis"/>
-        <origin xyz="$-0.1 0 0"/>
+        <origin xyz="-0.1 0 0"/>
     </joint>
     <link name="chassis">

Commit message: change 16:10p

File: description/robot_core.xacro (robot description, xacro)
@@ -1,5 +1,5 @@
 <?xml version="1.0"?>
 <robot xmlns:xacro="http://www.ros.org/wiki/xacro" >
-    <!-- <xacro:include filename="inertial_macros.xacro"/> -->
+    <xacro:include filename="inertial_macros.xacro"/>
     <material name="white">
         <color rgba="1 1 1 1" />
@@ -20,5 +20,5 @@
     <link name="base_link">
     </link>
-    <!-- toa do start-->
+    <!-- toa do start -->
     <link name="base_footprint">
     </link>
@@ -29,4 +29,23 @@
     </joint>
     <!-- khung xe-->
+    <link name="chassis">
+        <visual>
+            <origin xyz="0.15 0 0.075"/>
+            <geometry>
+                <box size="0.3 0.3 0.15"/>
+            </geometry>
+            <material name="white"/>
+        </visual>
+        <collision>
+            <origin xyz="0.15 0 0.075"/>
+            <geometry>
+                <box size="0.3 0.3 0.15"/>
+            </geometry>
+            <material name="white"/>
+        </collision>
+        <xacro:inertial_box mass="0.5" x="0.3" y="0.3" z="0.15">
+            <origin xyz="0.15 0 0.075" rpy="0.0 0.0 0.0">
+        </xacro:inertial_box>
+    </link>
     <joint name="chassis_joint" type="fixed">
         <parent link="base_link"/>
@@ -34,12 +53,74 @@
         <origin xyz="-0.1 0 0"/>
     </joint>
-    <link name="chassis">
+    <!-- banh xe trai-->
+    <link name="left_whell">
         <visual>
-            <origin xyz="0.15 0 0.074"/>
             <geometry>
-                <box size="0.3 0.3 0.15"/>
+                <cylinder radius="0.05" length="0.04"/>
             </geometry>
-            <material name="white"/>
+            <material name="blue"/>
         </visual>
+        <collision>
+            <geometry>
+                <cylinder radius="0.05" length="0.04"/>
+            </geometry>
+            <material name="blue"/>
+        </collision>
+        <xacro:inertial_cylinder mass="0.1" length="0.04" radius="0.05">
+            <origin xyz="0.0 0.0 0.0" rpy="0.0 0.0 0.0" />
+        </xacro:inertial_cylinder>
     </link>
+    <joint name="left_whell_joint" type="continuous">
+        <parent link="base_link"/>
+        <child link="left_whell"/>
+        <origin xyz="0 0.175 0" rpy="-${pi/2} 0 0 "/>
+          <axis xyz="0.0 0.0 1.0"/>
+    </joint>
+    <!-- banh xe phai -->
+    <link name="right_whell">
+        <visual>
+            <geometry>
+                <cylinder radius="0.05" length="0.04"/>
+            </geometry>
+            <material name="blue"/>
+        </visual>
+        <collision>
+            <geometry>
+                <cylinder radius="0.05" length="0.04"/>
+            </geometry>
+            <material name="blue"/>
+        </collision>
+        <xacro:inertial_cylinder mass="0.1" length="0.04" radius="0.05">
+            <origin xyz="0.0 0.0 0.0" rpy="0.0 0.0 0.0" />
+        </xacro:inertial_cylinder>
+    </link>
+    <joint name="right_whell_joint" type="continuous">
+        <parent link="base_link"/>
+        <child link="right_whell"/>
+        <origin xyz="0 -0.175 0" rpy="${pi/2} 0 0 "/>
+          <axis xyz="0.0 0.0 -1.0"/>
+    </joint>
+    <!-- banh xe da huong (choi lau nha) -->
+    <link name="caster_wheel">
+        <visual>
+            <geometry>
+                <sphere radius="0.05"/>
+            </geometry>
+            <material name="black"/>
+        </visual>
+        <collision>
+            <geometry>
+                <sphere radius="0.05"/>
+            </geometry>
+            <material name="black"/>
+        </collision>
+        <xacro:inertial_sphere mas="0.1" radius="0.05">
+            <origin xyz="0.0 0.0 0.0" rpy="0.0 0.0 0.0" />
+        </xacro:inertial_sphere>
+    </link>
+    <joint name="caster_wheel_joint" type="fixed">
+        <parent link="chassis"/>
+        <child link="caster_wheel"/>
+        <origin xyz="0.24 0 0"/>
+    </joint>
 </robot>

Commit message: change code 10h29p

File: description/robot_core.xacro (robot description, xacro)
@@ -45,5 +45,5 @@
         </collision>
         <xacro:inertial_box mass="0.5" x="0.3" y="0.3" z="0.15">
-            <origin xyz="0.15 0 0.075" rpy="0.0 0.0 0.0">
+            <origin xyz="0.15 0 0.075" rpy="0.0 0.0 0.0"/>
         </xacro:inertial_box>
     </link>
@@ -75,5 +75,5 @@
         <child link="left_whell"/>
         <origin xyz="0 0.175 0" rpy="-${pi/2} 0 0 "/>
-          <axis xyz="0.0 0.0 1.0"/>
+        <axis xyz="0.0 0.0 1.0"/>
     </joint>
     <!-- banh xe phai -->
@@ -99,5 +99,5 @@
         <child link="right_whell"/>
         <origin xyz="0 -0.175 0" rpy="${pi/2} 0 0 "/>
-          <axis xyz="0.0 0.0 -1.0"/>
+        <axis xyz="0.0 0.0 -1.0"/>
     </joint>
     <!-- banh xe da huong (choi lau nha) -->
@@ -115,5 +115,5 @@
             <material name="black"/>
         </collision>
-        <xacro:inertial_sphere mas="0.1" radius="0.05">
+        <xacro:inertial_sphere mass="0.1" radius="0.05">
             <origin xyz="0.0 0.0 0.0" rpy="0.0 0.0 0.0" />
         </xacro:inertial_sphere>

Commit message: add launch and gazebo

File: description/robot_core.xacro (robot description, xacro)
@@ -53,4 +53,8 @@
         <origin xyz="-0.1 0 0"/>
     </joint>
+    <!-- gazebo chassis -->
+    <gazebo reference="chassis">
+        <material>Gazebo/white</material>
+    </gazebo>
     <!-- banh xe trai-->
     <link name="left_whell">
@@ -77,4 +81,8 @@
         <axis xyz="0.0 0.0 1.0"/>
     </joint>
+    <!-- Gazebo banh xe trai -->
+    <gazebo reference="left_wheel">
+        <material>Gazebo/blue</material>
+    </gazebo>
     <!-- banh xe phai -->
     <link name="right_whell">
@@ -101,4 +109,8 @@
         <axis xyz="0.0 0.0 -1.0"/>
     </joint>
+    <!-- Gazebo banh xe phai -->
+    <gazebo reference="right_wheel">
+        <material>Gazebo/Blue</material>
+    </gazebo>
     <!-- banh xe da huong (choi lau nha) -->
     <link name="caster_wheel">
@@ -124,3 +136,7 @@
         <origin xyz="0.24 0 0"/>
     </joint>
+    <!-- Gazebo banh xe da huong -->
+    <gazebo reference="caster_wheel">
+        <material>Gazebo/Black</material>
+    </gazebo>
 </robot>
