Commit message: change 15h32p

File: description/robot.urdf.xacro (robot description, xacro)
@@ -2,3 +2,4 @@
 <robot xmlns:xacro="http://www.ros.org/wiki/xacro"  name="robot">
     <xacro:include filename="robot_core.xacro" />
+    <!-- <xacro:include filename="gazebo_control.xacro" /> -->
 </robot>

File: description/robot_core.xacro (robot description, xacro)
@@ -21,11 +21,11 @@
     </link>
     <!-- toa do start -->
-    <link name="base_footprint">
-    </link>
-    <joint name="base_footprint_joint" type="fixed">
+    <!-- <link name="base_footprint">
+    </link> -->
+    <!-- <joint name="base_footprint_joint" type="fixed">
         <parent link="base_link"/>
         <child link="base_footprint"/>
         <origin xyz="0 0 0" rpy="0 0 0"/>
-    </joint>
+    </joint> -->
     <!-- khung xe-->
     <link name="chassis">
@@ -58,5 +58,5 @@
     </gazebo>
     <!-- banh xe trai-->
-    <link name="left_whell">
+    <link name="left_wheel">
         <visual>
             <geometry>
@@ -75,7 +75,7 @@
         </xacro:inertial_cylinder>
     </link>
-    <joint name="left_whell_joint" type="continuous">
+    <joint name="left_wheel_joint" type="continuous">
         <parent link="base_link"/>
-        <child link="left_whell"/>
+        <child link="left_wheel"/>
         <origin xyz="0 0.175 0" rpy="-${pi/2} 0 0 "/>
         <axis xyz="0.0 0.0 1.0"/>
@@ -83,8 +83,10 @@
     <!-- Gazebo banh xe trai -->
     <gazebo reference="left_wheel">
-        <material>Gazebo/blue</material>
+        <material>
+            Gazebo/Blue
+        </material>
     </gazebo>
     <!-- banh xe phai -->
-    <link name="right_whell">
+    <link name="right_wheel">
         <visual>
             <geometry>
@@ -103,7 +105,7 @@
         </xacro:inertial_cylinder>
     </link>
-    <joint name="right_whell_joint" type="continuous">
+    <joint name="right_wheel_joint" type="continuous">
         <parent link="base_link"/>
-        <child link="right_whell"/>
+        <child link="right_wheel"/>
         <origin xyz="0 -0.175 0" rpy="${pi/2} 0 0 "/>
         <axis xyz="0.0 0.0 -1.0"/>
@@ -111,5 +113,7 @@
     <!-- Gazebo banh xe phai -->
     <gazebo reference="right_wheel">
-        <material>Gazebo/Blue</material>
+        <material>
+            Gazebo/Blue
+        </material>
     </gazebo>
     <!-- banh xe da huong (choi lau nha) -->
@@ -139,4 +143,6 @@
     <gazebo reference="caster_wheel">
         <material>Gazebo/Black</material>
+        <mu1 value = "0.001"/>
+        <mu2 value = "0.001"/>
     </gazebo>
 </robot>

Commit message: confirm 16h26

File: description/robot.urdf.xacro (robot description, xacro)
@@ -2,4 +2,4 @@
 <robot xmlns:xacro="http://www.ros.org/wiki/xacro"  name="robot">
     <xacro:include filename="robot_core.xacro" />
-    <!-- <xacro:include filename="gazebo_control.xacro" /> -->
+    <xacro:include filename="gazebo_control.xacro" />
 </robot>

File: description/robot_core.xacro (robot description, xacro)
@@ -21,11 +21,11 @@
     </link>
     <!-- toa do start -->
-    <!-- <link name="base_footprint">
-    </link> -->
-    <!-- <joint name="base_footprint_joint" type="fixed">
+    <link name="base_footprint">
+    </link>
+    <joint name="base_footprint_joint" type="fixed">
         <parent link="base_link"/>
         <child link="base_footprint"/>
         <origin xyz="0 0 0" rpy="0 0 0"/>
-    </joint> -->
+    </joint>
     <!-- khung xe-->
     <link name="chassis">
